File: tcspc_eagleproj/tcspc/tcspc.sch (EAGLE design)
At the start: 86 parts, among them U1 THS788, U2 MCP4725, U3 ADCMP582, U4 LT6003_SOT23-5, U5 LT6003_SOT23-5, X1 SMA

Commit message: turned the frontend into a useful designblock, ready to be pased all over the tcspc board
Parts:
- removed C1, C2: 10pF, tcspc_lib:CAP_0402
- removed C10, C11, C12, C13, C15, C17, C19, C21, C23, C25, C27, C29, C3, C31, C33, C35, C37, C39, C4, C41, C43, C45, C53, C54, C55, C6, C7, C8, C9: .1uF, tcspc_lib:CAP_0402
- removed C14, C16, C18, C20, C22, C24, C26, C28, C30, C32, C34, C36, C38, C40, C42, C44, C46, C52: 10nF, tcspc_lib:CAP_0402
- removed C47: .1uF, tcspc_lib:CAP_0603
- removed C48, C49, C50, C51: 1uF, tcspc_lib:CAP_0603
- removed C5: 10uF, tcspc_lib:CAP_0402
- removed G1: 200MHz, tcspc_lib:SIT5021
- removed Q1: (no value), jack_semi:BJT_NPN
- removed R1, R2: 50, tcspc_lib:RES_0402
- removed R10, R11, R12, R13: (no value), tcspc_lib:RES_0402
- removed R14, R6, R9: 0, tcspc_lib:RES_0402
- removed R15: 210, tcspc_lib:RES_0402
- removed R16: 100, tcspc_lib:RES_0402
- removed R17, R18, R19, R20, R21, R22, R23: DNP, tcspc_lib:RES_0402
- removed R3, R4, R5: 1k, tcspc_lib:RES_0402
- removed R7, R8: 2.2k, tcspc_lib:RES_0402
- removed U1: THS788, tcspc_lib:THS788
- removed U2: MCP4725, tcspc_lib:MCP4725
- removed U3: ADCMP582, tcspc_lib:ADCMP582
- removed U4, U5: LT6003_SOT23-5, tcspc_lib:LT6003_SOT23-5
- removed X1: SMA, tcspc_lib:SMA
Connections:
- removed net !TMU_DOUT_A: U1.!RDATA-A
- removed net !TMU_IN_A: U1.!EVENT-A
- removed net !TMU_IN_B: U1.!EVENT-B
- removed net !TMU_IN_C: U1.!EVENT-C
- removed net !TMU_IN_D: U1.!EVENT-D
- removed net GND: C10.2, C11.2, C12.2, C13.2, C14.2, C15.2, C16.2, C17.2, C18.2, C19.2, C20.2, C21.2, C22.2, C23.2, C24.2, C25.2, C26.2, C27.2, C28.2, C29.2, C3.2, C30.2, C31.2, C32.2, C33.2, C34.2, C35.2, C36.2, C37.2, C38.2, C39.2, C4.2, C40.2, C41.2, C42.2, C43.2, C44.2, C45.2, C46.2, C47.2, C48.2, C49.2, C5.2, C50.2, C51.2, C52.1, C53.2, C54.2, C55.2, C6.2, C7.1, C8.2, C9.2, G1.GND, R1.2, R12.2, R13.2, R15.2, R18.2, R2.2, R20.2, R5.2, R9.1, U1.GND, U2.A0, U2.VSS, U3.GND, U3.VTN, U5.IN+, X1.GND
- removed net N$1: G1.OUT-, U1.!MCLK
- removed net N$10: U1.TEMP
- removed net N$11: U1.OT_ALRM
- removed net N$12: R3.1, R4.2, U4.IN-
- removed net N$13: R14.1, R3.2, U4.OUT
- removed net N$14: U1.!RESET
- removed net N$15: U1.HDATA
- removed net N$16: U1.HCLK
- removed net N$17: U1.!HSTROBE
- removed net N$18: U3.VN, X1.1
- removed net N$19: R7.2, U2.SCL
- removed net N$2: G1.OUT+, U1.MCLK
- removed net N$20: R8.2, U2.SDA
- removed net N$21: U1.!RSTROBE-D
- removed net N$22: U1.RSTROBE-D
- removed net N$23: U1.!RSTROBE-C
- removed net N$24: U1.RSTROBE-C
- removed net N$25: U1.!RSTROBE-B
- removed net N$26: U1.RSTROBE-B
- removed net N$27: U1.!RSTROBE-A
- removed net N$28: U1.RSTROBE-A
- removed net N$29: U1.!RCLK
- removed net N$3: C2.1, R2.1, U3.!Q
- removed net N$30: U1.RCLK
- removed net N$31: U1.!RDATA-D
- removed net N$32: U1.RDATA-D
- removed net N$33: U1.!RDATA-C
- removed net N$34: U1.RDATA-C
- removed net N$35: U1.!RDATA-B
- removed net N$36: U1.RDATA-B
- removed net N$37: C52.2, R14.2, U3.VP
- removed net N$38: R17.2, R18.1, U3.VTT
- removed net N$39: R15.1, R19.2, U3.LE
- removed net N$4: C1.2, R10.2, R12.1
- removed net N$41: R16.2, R20.1, U3.!LE
- removed net N$42: Q1.C, U3.HYS
- removed net N$43: Q1.B, U5.OUT
- removed net N$45: C55.1, R22.2, R23.1, U5.IN-
- removed net N$46: R22.1
- removed net N$47: Q1.E, R21.1, R23.2
- removed net N$5: C2.2, R11.2, R13.1
- removed net N$6: C1.1, R1.1, U3.Q
- removed net N$7: R9.2, U3.VTP
- removed net N$8: R6.1, U2.OUT
- removed net N$9: C3.1, R5.1, R6.2, U4.IN+
- removed net PP_N3V3_ANALOG: C53.1, C7.2, C8.1, R21.2, U3.VEE, U4.V-, U5.V-
- removed net PP_P3V3: C13.1, C14.1, C15.1, C16.1, C17.1, C18.1, C19.1, C20.1, C21.1, C22.1, C23.1, C24.1, C25.1, C26.1, C27.1, C28.1, C29.1, C30.1, C31.1, C32.1, C33.1, C34.1, C35.1, C36.1, C37.1, C38.1, C39.1, C40.1, C41.1, C42.1, C43.1, C44.1, C45.1, C46.1, C47.1, C48.1, C49.1, C50.1, C51.1, G1.VDD, U1.VCC
- removed net PP_P3V3_ANALOG: C10.1, C11.1, C4.1, C5.1, C54.1, C6.1, C9.1, R4.1, R7.1, R8.1, U2.VDD, U3.VCCI, U4.V+, U5.V+
- removed net PP_P3V3_DIGITAL: C12.1, R10.1, R11.1, R16.1, R17.1, R19.1, U3.VCCO
- removed net TMU_DOUT_A: U1.RDATA-A
- removed net TMU_IN_A: U1.EVENT-A
- removed net TMU_IN_B: U1.EVENT-B
- removed net TMU_IN_C: U1.EVENT-C
- removed net TMU_IN_D: U1.EVENT-D
Other:
- note removed: "100 Ohm Differential Transmission Line"
- note removed: "100_OHM_DIFF"
- note removed: "50 Ohm Single Ended Transmission Line"
- note removed: "50_OHM_SE"
- note removed: "I2C Control Input"
- note removed: "LVDS TMU INPUT"
- note removed: "Signal"
- note removed: "Signal Input"
- note removed: "Threshold"
- note removed: "Threshold Control DAC"
- note removed: "To disable latching, LE should be at 1.7V and !LE! at 2.5V Here, the current across the internal 100 ohm termination between LE and !LE! needs to be 8mA."

Commit message: small tweaks to the dbl so that I could start putting four of them onto the main board, and then I did just that.
Parts:
- added C10, C18, C19, C20, C28, C29, C30, C38, C39, C40, C8, C9: 100nF, tcspc_lib:CAP_0402
- added C16, C17, C26, C27, C36, C37, C6, C7: 10nF, tcspc_lib:CAP_0402
- added R13, R21, R29, R5: 50, tcspc_lib:RES_0402
- added R14, R22, R30, R6: 1k, tcspc_lib:RES_0402
- added R15, R23, R31, R7: 90.2k, tcspc_lib:RES_0402
- added R16, R24, R32, R8: 55k, tcspc_lib:RES_0402
- added U2, U4, U6, U8: AD8465, tcspc_lib:AD8465
- added X2, X4, X6, X8: SMA, tcspc_lib:SMA
Connections:
- new net CHA_HYS_SET: R7.1
- new net CHA_LE/HYS: R7.2, R8.1, U2.LE/HYS
- new net CHA_OUT_N: U2.!Q
- new net CHA_OUT_P: U2.Q
- new net CHA_SIG_IN: R5.1, U2.VN, X2.1
- new net CHA_THRESH: C10.1, R6.2, U2.VP
- new net CHA_THRESH_SET: R6.1
- new net CHB_HYS_SET: R15.1
- new net CHB_LE/HYS: R15.2, R16.1, U4.LE/HYS
- new net CHB_OUT_N: U4.!Q
- new net CHB_OUT_P: U4.Q
- new net CHB_SIG_IN: R13.1, U4.VN, X4.1
- new net CHB_THRESH: C20.1, R14.2, U4.VP
- new net CHB_THRESH_SET: R14.1
- new net CHC_HYS_SET: R23.1
- new net CHC_LE/HYS: R23.2, R24.1, U6.LE/HYS
- new net CHC_OUT_N: U6.!Q
- new net CHC_OUT_P: U6.Q
- new net CHC_SIG_IN: R21.1, U6.VN, X6.1
- new net CHC_THRESH: C30.1, R22.2, U6.VP
- new net CHC_THRESH_SET: R22.1
- new net CHD_HYS_SET: R31.1
- new net CHD_LE/HYS: R31.2, R32.1, U8.LE/HYS
- new net CHD_OUT_N: U8.!Q
- new net CHD_OUT_P: U8.Q
- new net CHD_SIG_IN: R29.1, U8.VN, X8.1
- new net CHD_THRESH: C40.1, R30.2, U8.VP
- new net CHD_THRESH_SET: R30.1
- new net GND: C10.2, C16.2, C17.2, C18.2, C19.2, C20.2, C26.2, C27.2, C28.2, C29.2, C30.2, C36.2, C37.2, C38.2, C39.2, C40.2, C6.2, C7.2, C8.2, C9.2, R13.2, R16.2, R21.2, R24.2, R29.2, R32.2, R5.2, R8.2, U2.SDN, U2.VEE, U4.SDN, U4.VEE, U6.SDN, U6.VEE, U8.SDN, U8.VEE, X2.GND, X4.GND, X6.GND, X8.GND
- new net PP_P3V3_ANALOG: C16.1, C18.1, C26.1, C28.1, C36.1, C38.1, C6.1, C8.1, U2.VCCI, U4.VCCI, U6.VCCI, U8.VCCI
- new net PP_P3V3_DIGITAL: C17.1, C19.1, C27.1, C29.1, C37.1, C39.1, C7.1, C9.1, U2.VCCO, U4.VCCO, U6.VCCO, U8.VCCO
Other:
- note added: "100_OHM_DIFF"
- note added: "50 Ohm Single Ended Transmission Line"
- note added: "50_OHM_SE"

Commit message: created an FPGA device in the library, stuck it on the board and hooked up the various power pins to their nets. I also added the linear postregs and DAC to the schematic, and did some power calcs.
Parts:
- added C1, C2, C21, C25, C33, C34: 100nF, tcspc_lib:CAP_0402
- added C11, C12, C22, C24: 10uF, tcspc_lib:CAP_0603
- added C13, C14, C15, C23, C3, C31, C4, C5: 10nF, tcspc_lib:CAP_0402
- added C32, C35, C41: 10uF, tcspc_lib:CAP_0402
- added FPGA1: XEM7310, tcspc_lib:XEM7310
- added R1, R3: 17.8k, tcspc_lib:RES_0402
- added R2, R4: 10k, tcspc_lib:RES_0402
- added U1: AD53X8, tcspc_lib:AD53X8
- added VR1, VR2: (no value), tcspc_lib:TPS7A49
Connections:
- new net DAC_!LDAC!: U1.!LDAC
- new net DAC_!SYNC!: U1.!SYNC
- new net DAC_DIN: U1.DIN
- new net DAC_SCLK: U1.SCLK
- new net FPGA_SYS_CLK_MC1: FPGA1-MC1-E.P4
- new net FPGA_SYS_CLK_MC2: FPGA1-MC2-O.P6
- new net FPGA_TCK: FPGA1-MC2-O.P3
- new net FPGA_TDI: FPGA1-MC2-O.P5
- new net FPGA_TDO: FPGA1-MC2-E.P4
- new net FPGA_TMS: FPGA1-MC2-O.P4
- new net FPGA_VCCO_MC1: FPGA1-MC1-E.P18, FPGA1-MC1-E.P28
- new net FPGA_VCCO_MC2: FPGA1-MC2-O.P18, FPGA1-MC2-O.P28
- new net FPGA_XADC_VN: FPGA1-MC1-E.P5
- new net FPGA_XADC_VP: FPGA1-MC1-E.P6
- new net N$1: C1.1, C11.1, C13.1, VR1.EN, VR1.IN
- new net N$10: C23.2, R3.2, R4.1, VR2.FB
- new net N$11: U1.VOUT_C
- new net N$12: U1.VOUT_D
- new net N$13: U1.VOUT_E
- new net N$14: U1.VOUT_F
- new net N$15: U1.VOUT_G
- new net N$16: U1.VOUT_H
- new net N$2: U1.VOUT_A
- new net N$3: C4.2, R1.2, R2.1, VR1.FB
- new net N$4: C3.1, VR1.NR
- new net N$7: C15.1, C21.1, C22.1, VR2.EN, VR2.IN
- new net N$8: C14.1, VR2.NR
- new net N$9: U1.VOUT_B
- new net PP_P1V0_FPGA: FPGA1-MC1-E.P2, FPGA1-MC1-E.P3
- new net PP_P1V8_FPGA: FPGA1-MC1-O.P4
- new net PP_P3V3_FPGA: FPGA1-MC1-O.P5, FPGA1-MC1-O.P6, FPGA1-MC1-O.P7, FPGA1-MC2-E.P1, FPGA1-MC2-E.P2, FPGA1-MC2-E.P3
- new net PP_VCCBATT_FPGA: FPGA1-MC2-O.P2
- new net PP_VDCIN_FPGA: FPGA1-MC1-O.P1, FPGA1-MC1-O.P2, FPGA1-MC1-O.P3
- net GND: now also C1.2, C11.2, C12.2, C13.2, C14.2, C15.2, C2.2, C21.2, C22.2, C24.2, C25.2, C3.2, C31.2, C32.2, C33.2, C34.2, C35.2, C41.2, C5.2, FPGA1-MC1-E.P1, FPGA1-MC1-E.P39, FPGA1-MC1-E.P40, FPGA1-MC1-E.P7, FPGA1-MC1-O.P18, FPGA1-MC1-O.P28, FPGA1-MC2-E.P18, FPGA1-MC2-E.P28, FPGA1-MC2-E.P39, FPGA1-MC2-E.P40, FPGA1-MC2-E.P7, FPGA1-MC2-O.P1, FPGA1-MC2-O.P7, R2.2, R4.2, U1.GND, VR1.GND, VR2.GND
- net PP_P3V3_ANALOG: now also C12.1, C2.1, C32.1, C33.1, C4.1, C41.1, C5.1, R1.1, U1.VREF_ABCD, U1.VREF_EFGH, VR1.OUT
- net PP_P3V3_DIGITAL: now also C23.1, C24.1, C25.1, C31.1, C34.1, C35.1, R3.1, U1.V_DD, VR2.OUT
