File: tcspc_eagleproj/tcspc/frontend.sch (EAGLE design)
At the start: 100 parts, among them Q2 ALD1101SAL, U1 DS90LV028AQ, U3 ADCMP582, U4 LT6003_SOT23-5, U5 LT6003_SOT23-5, U6 AD53X8, X1 SMA, X2 SMA

Commit message: Added and have been working on the THS788 carrier board for a while without committing it
Parts:
- removed C52: 10nF, tcspc_lib:CAP_0402
- removed C53, C54, C55: 100nF, tcspc_lib:CAP_0402
- removed R27: 10k, tcspc_lib:RES_0402
- removed U6: AD53X8, tcspc_lib:AD53X8
- added C35, C37: 100nF, tcspc_lib:CAP_0402
- added C36, C38: 10nF, tcspc_lib:CAP_0402
- added R8: 50, tcspc_lib:RES_0402
- added U2: ADCMP582, tcspc_lib:ADCMP582
- C1, C2: value 10pF -> 100nF
- C14, C15, C17, C22, C24, C25: value 10nF -> 100nF
- C18, C21, C29, C30, C8: value 100nF -> 10nF
- C3, C4: value 100nF -> 10pF
- C31, C33: value 10uF -> 100nF
- C32: value 10uF -> 10nF
- C34, C5: value 100uF -> 10nF
- Q1: value (none) -> ALD1101SAL; device tcspc_lib:MOSFET_P-CHANNEL_SOT23-3 -> tcspc_lib:ALD1101SAL
- Q2: value ALD1101SAL -> (none); device tcspc_lib:ALD1101SAL -> tcspc_lib:MOSFET_P-CHANNEL_SOT23-3
- R1: value 50 -> 100
- R10: value 3.2k -> 1.8k
- R11: value 3.2k -> 50
- R12: value 1.8k -> 3.2k
- R15: value 210 -> 0
- R16: value 100 -> 5500
- R17, R18, R19, R20: value DNP -> 1k
- R2: value 50 -> DNP
- R21: value 5500 -> 17.8k
- R23: value 10k -> 17.8k
- R24, R26: value 17.8k -> 10k
- R3: value 1k -> 210
- R4, R6: value 1k -> DNP
- R5: value 1k -> 100
- R7: value 100 -> DNP
- R9: value 0 -> 3.2k
- TP1: value DAC_SCLK -> GND
- TP10: value DAC_OUT_A -> HYS_PIN
- TP11: value DAC_OUT_B -> MIRROR_GATE
- TP12: value DAC_OUT_E -> HYS_RSENSE
- TP13: value DAC_OUT_H -> P3V3A
- TP14: value THRESH -> P3V3D
- TP15: value HYS_RSENSE -> N3V3A
- TP16: value MIRROR_GATE -> DAC_OUT_H
- TP17: value HYS_PIN -> DAC_OUT_E
- TP18: value !ECL_OUT -> DAC_!LDAC!; device tcspc_lib:TESTPOINT_PAD -> tcspc_lib:TESTPOINT_A
- TP19: value ECL_OUT -> DAC_!SYNC!; device tcspc_lib:TESTPOINT_PAD -> tcspc_lib:TESTPOINT_A
- TP2: value DAC_!SYNC! -> !ECL_OUT; device tcspc_lib:TESTPOINT_A -> tcspc_lib:TESTPOINT_PAD
- TP20: value LVDS_OUT -> DAC_SCLK; device tcspc_lib:TESTPOINT_PAD -> tcspc_lib:TESTPOINT_A
- TP21: value !LVDS_OUT -> DAC_DIN; device tcspc_lib:TESTPOINT_PAD -> tcspc_lib:TESTPOINT_A
- TP3: value DAC_DIN -> !LVDS_OUT; device tcspc_lib:TESTPOINT_A -> tcspc_lib:TESTPOINT_PAD
- TP4: value DAC_!LDAC! -> ECL_OUT; device tcspc_lib:TESTPOINT_A -> tcspc_lib:TESTPOINT_PAD
- TP5: value P3V3D -> LVDS_OUT; device tcspc_lib:TESTPOINT_A -> tcspc_lib:TESTPOINT_PAD
- TP6: value P3V3A -> GND
- TP7: value N3V3A -> DAC_OUT_A
- TP8: value GND -> DAC_OUT_B
- TP9: value GND -> THRESH
- U3: value ADCMP582 -> LT6003_SOT23-5; device tcspc_lib:ADCMP582 -> tcspc_lib:LT6003_SOT23-5
- U5: value LT6003_SOT23-5 -> AD53X8; device tcspc_lib:LT6003_SOT23-5 -> tcspc_lib:AD53X8
Connections:
- net !CHA_LVDS_OUT: now also C3.2, R1.2, R10.1, R9.2, TP3.TP; no longer C2.2, R11.2, R13.1, R7.2, TP21.TP
- net CHA_HYS_SET: now also R20.1, TP8.TP, U5.VOUT_B; no longer R6.1, TP11.TP, U6.VOUT_B
- net CHA_LVDS_OUT: now also C4.2, R1.1, R12.2, R13.1, TP5.TP; no longer C1.2, R10.2, R12.1, R7.1, TP20.TP
- net CHA_THRESH_SET: now also R17.1, TP7.TP, U5.VOUT_A; no longer R5.1, TP10.TP, U6.VOUT_A
- net GND: now also C1.2, C10.1, C15.2, C2.2, C20.2, C26.2, C35.2, C36.2, C37.2, C38.2, C5.1, C7.2, R10.2, R11.2, R14.1, R24.1, R26.1, R3.2, R4.2, R8.2, TP1.TP, TP6.TP, U2.GND, U2.VTN, U5.GND; no longer C10.2, C28.2, C29.2, C3.2, C30.2, C4.2, C5.2, C52.1, C53.2, C54.2, C55.2, C7.1, R1.2, R12.2, R15.2, R18.2, R20.2, R23.1, R27.1, R9.1, TP8.TP, TP9.TP, U3.GND, U3.VTN, U6.GND
- net N$1: now also Q2.S, R16.2, TP12.TP, U3.IN-; no longer Q1.S, R21.2, TP15.TP, U5.IN-
- net N$10: now also Q2.G, U3.OUT; no longer Q1.G, U5.OUT
- net N$11: now also TP16.TP, U5.VOUT_H; no longer TP13.TP, U6.VOUT_H
- net N$12: now also R18.1, R19.2; no longer R3.1, R4.2
- net N$13: now also R15.1, R18.2, TP9.TP; no longer R14.1, R3.2, TP14.TP
- net N$16: now also C36.1; no longer C25.1
- net N$17: now also C17.1, R20.2, U3.IN+; no longer C55.1, R6.2, U5.IN+
- net N$18: now also U2.VN; no longer U3.VN
- net N$19: now also C34.1; no longer C14.1
- net N$2: now also Q1_A.D, Q1_A.G, Q1_B.G, Q2.D, TP11.TP; no longer Q1.D, Q2_A.D, Q2_A.G, Q2_B.G, TP16.TP
- net N$21: now also C29.2, R22.2, R25.2; no longer C26.2, R26.2, R27.2
- net N$25: now also C38.1; no longer C19.1
- net N$3: now also C3.1, R8.1, TP2.TP, U2.!Q; no longer C2.1, R2.1, TP18.TP, U3.!Q
- net N$37: now also C5.2, R15.2, U2.VP; no longer C52.2, R14.2, U3.VP
- net N$38: now also R4.1, R7.2, U2.VTT; no longer R17.2, R18.1, U3.VTT
- net N$39: now also R3.1, R6.2, U2.LE; no longer R15.1, R19.2, U3.LE
- net N$4: now also C30.2, R23.2, R26.2; no longer C20.2, R24.2, R25.2
- net N$41: now also R2.1, R5.2, U2.!LE; no longer R16.2, R20.1, U3.!LE
- net N$42: now also Q1_B.D, TP10.TP, U2.HYS; no longer Q2_B.D, TP17.TP, U3.HYS
- net N$5: now also C28.2, R21.2, R24.2; no longer C15.2, R22.2, R23.2
- net N$6: now also C4.1, R11.1, TP4.TP, U2.Q; no longer C1.1, R1.1, TP19.TP, U3.Q
- net N$7: now also R14.2, U2.VTP; no longer R9.2, U3.VTP
- net N$8: now also TP17.TP, U5.VOUT_E; no longer TP12.TP, U6.VOUT_E
- net N$9: now also C13.1, R17.2; no longer C3.1, R5.2
- net PP_N3V3_ANALOG: now also C10.2, C12.1, C14.1, C15.1, C24.1, C30.1, Q1_A.S, Q1_B.S, R23.1, TP15.TP, U2.VEE, U3.V-; no longer C21.1, C22.1, C4.1, C53.1, C7.2, C8.1, Q2_A.S, Q2_B.S, R24.1, TP7.TP, U3.VEE, U5.V-
- net PP_N5V_VIN: now also C37.1; no longer C18.1
- net PP_P3V3_ANALOG: now also C11.1, C18.1, C2.1, C22.1, C26.1, C27.1, C28.1, C31.1, R16.1, R19.1, TP13.TP, U2.VCCI, U3.V+, U5.VREF_ABCD, U5.VREF_EFGH; no longer C10.1, C15.1, C17.1, C33.1, C34.1, C5.1, C54.1, C6.1, R22.1, R4.1, TP6.TP, U3.VCCI, U5.V+, U6.VREF_ABCD, U6.VREF_EFGH
- net PP_P3V3_DIGITAL: now also C1.1, C19.1, C21.1, C25.1, C29.1, C6.1, C7.1, C8.1, R12.1, R22.1, R5.1, R6.1, R7.1, R9.1, TP14.TP, U2.VCCO, U5.V_DD; no longer C11.1, C12.1, C24.1, C26.1, C27.1, C28.1, C30.1, C31.1, R10.1, R11.1, R16.1, R17.1, R19.1, R26.1, TP5.TP, U3.VCCO, U6.V_DD
- net PP_P5V_VIN: now also C33.1, C35.1; no longer C13.1, C29.1
- net T/H_DAC_!LDAC!: now also TP18.TP, U5.!LDAC; no longer TP4.TP, U6.!LDAC
- net T/H_DAC_!SYNC!: now also TP19.TP, U5.!SYNC; no longer TP2.TP, U6.!SYNC
- net T/H_DAC_DIN: now also TP21.TP, U5.DIN; no longer TP3.TP, U6.DIN
- net T/H_DAC_SCLK: now also TP20.TP, U5.SCLK; no longer TP1.TP, U6.SCLK
